File: redPad/redPad.kicad_sch (KiCad schematic)
At the start: 26 parts, among them SW1 RotaryEncoder_Switch_MP, SW2 RotaryEncoder_Switch_MP

Commit message: Avance en teclado
Parts:
- removed SW1, SW2: RotaryEncoder_Switch_MP, Rotary_Encoder:RotaryEncoder_Alps_EC11E-Switch_Vertical_H20mm_MountingHoles, symbol Device:RotaryEncoder_Switch_MP
- added BT1: Battery, Connector_JST:JST_ACH_BM01B-ACHSS-A-GAN-ETF_1x01-1MP_P1.20mm_Vertical, symbol Device:Battery
- added D13, D14: Diode, Diode_SMD:D_SOD-123, symbol ScottoKeebs:Placeholder_Diode
- added J1: OLED_128x32, ScottoKeebs_Components:OLED_128x32, symbol ScottoKeebs:OLED_128x32
- added SW1, SW2: RotaryEncoder_Switch, Rotary_Encoder:RotaryEncoder_Alps_EC11E-Switch_Vertical_H20mm, symbol Device:RotaryEncoder_Switch
- added SW3: SW_Push, ScottoKeebs_Components:Button_TL3342, symbol Switch:SW_Push
- added SW4: Switch, ScottoKeebs_Components:Switch_MSK12C02, symbol ScottoKeebs:Placeholder_Switch
- added SuperMini-NRF1: ~, RedComponents:SuperMini NRF52840, symbol SuperMini:SuperMini NRF52840
- D1, D10, D11, D12, D2, D3, D4, D5, D6, D7, D8, D9: footprint (none) -> Diode_SMD:D_SOD-123
- S1, S10, S11, S12, S2, S3, S4, S5, S6, S7, S8, S9: footprint (none) -> ScottoKeebs_Hotswap:Hotswap_MX_1.00u
Connections:
- net ROW 0: now reaches D1.1 (K), D2.1 (K), D3.1 (K), D4.1 (K)
- net ROW 0: now also SuperMini-NRF1.24 (P1.11/D14)
- net ROW 1: now reaches D5.1 (K), D6.1 (K), D7.1 (K), D8.1 (K)
- net ROW 1: now also SuperMini-NRF1.23 (P1.13/D15)
- net COL 2: now reaches S11.1, S3.1, S7.1
- net COL 2: now also SuperMini-NRF1.9 (P0.24/D5)
- net COL 3: now reaches S12.1, S4.1, S8.1
- net COL 3: now also SuperMini-NRF1.8 (P0.22/D4)
- net COL 1: now reaches S10.1, S2.1, S6.1
- net COL 1: now also SW2.S1, SuperMini-NRF1.10 (P1.00/D6)
- net ROW 2: now reaches D10.1 (K), D11.1 (K), D12.1 (K), D9.1 (K)
- net ROW 2: now also SuperMini-NRF1.22 (P1.15/D18)
- net COL 0: now reaches S1.1, S5.1, S9.1
- net COL 0: now also SW1.S1, SuperMini-NRF1.11 (P0.11/D7)
- new net: BT1.1 (+), SW4.1
- new net: D14.2 (A), SW2.S2
- new net: D13.2 (A), SW1.S2
- new net BAT +: SW4.2, SuperMini-NRF1.14 (B+)
- new net BAT -: BT1.2 (-), SuperMini-NRF1.1 (B-/GND)
- new net ENC 1: SW1.B, SuperMini-NRF1.20 (P0.29/D20)
- new net ENC 2: SW1.A, SuperMini-NRF1.19 (P0.31/D21)
- new net ENC 3: SW2.B, SuperMini-NRF1.2 (P0.06/D1)
- new net ENC 4: SW2.A, SuperMini-NRF1.3 (P0.08/D0)
- new net GND: J1.1 (GND), SW1.C, SW2.C, SW3.2, SuperMini-NRF1.16 (GND), SuperMini-NRF1.4 (GND), SuperMini-NRF1.5 (GND)
- new net OLED SCL: J1.3 (SCL), SuperMini-NRF1.6 (P0.17/D2)
- new net OLED SDA: J1.4 (SDA), SuperMini-NRF1.7 (P0.20/D3)
- new net ROW 3: D13.1 (K), D14.1 (K), SuperMini-NRF1.21 (P0.02/D19)
- new net RST: SW3.1, SuperMini-NRF1.17 (RST)
- new net VCC: J1.2 (VCC), SuperMini-NRF1.18 (VCC)
Other:
- moved on the sheet: D1, D10, D11, D12, D2, D3, D4, D5, D6, D7, D8, D9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

Commit message: Version 1.0 finalizada
Parts:
- BT1: footprint Connector_JST:JST_ACH_BM01B-ACHSS-A-GAN-ETF_1x01-1MP_P1.20mm_Vertical -> Connector_JST:JST_EH_S2B-EH_1x02_P2.50mm_Horizontal
- SW3: footprint ScottoKeebs_Components:Button_TL3342 -> RedComponents:SW TS-B003-Y
Connections:
- net BAT -: now also BT1.1 (+); no longer BT1.2 (-)
- net COL 0: now also SuperMini-NRF1.8 (P0.22/D4); no longer SuperMini-NRF1.11 (P0.11/D7)
- net COL 1: now also SuperMini-NRF1.9 (P0.24/D5); no longer SuperMini-NRF1.10 (P1.00/D6)
- net COL 2: now also SuperMini-NRF1.10 (P1.00/D6); no longer SuperMini-NRF1.9 (P0.24/D5)
- net COL 3: now also SuperMini-NRF1.11 (P0.11/D7); no longer SuperMini-NRF1.8 (P0.22/D4)
- net at SW4.1: now also BT1.2 (-); no longer BT1.1 (+)
Other:
- moved on the sheet: BT1
Changed lines of the file:
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@@
 	(wire
 		(pts
-			(xy 181.61 86.36) (xy 185.42 86.36)
+			(xy 63.5 76.2) (xy 63.5 101.6)
 		)
 		(stroke
@@
 	(wire
 		(pts
-			(xy 63.5 76.2) (xy 63.5 101.6)
+			(xy 165.1 129.54) (xy 175.26 129.54)
 		)
 		(stroke
@@
 	(wire
 		(pts
-			(xy 165.1 129.54) (xy 175.26 129.54)
+			(xy 128.27 142.24) (xy 190.5 142.24)
 		)
 		(stroke
@@
 	(wire
 		(pts
-			(xy 128.27 142.24) (xy 190.5 142.24)
+			(xy 181.61 78.74) (xy 185.42 78.74)
 		)
 		(stroke
@@
 	(wire
 		(pts
+			(xy 181.61 81.28) (xy 185.42 81.28)
+		)
+		(stroke
+			(width 0)
+			(type default)
+		)
+	)
+	(wire
+		(pts
 			(xy 125.73 63.5) (xy 139.7 63.5)
 		)
@@
 	(wire
 		(pts
+			(xy 181.61 83.82) (xy 185.42 83.82)
+		)
+		(stroke
+			(width 0)
+			(type default)
+		)
+	)
+	(wire
+		(pts
 			(xy 101.6 76.2) (xy 101.6 101.6)
 		)
@@
 	(wire
 		(pts
-			(xy 88.9 158.75) (xy 88.9 157.48)
+			(xy 181.61 86.36) (xy 185.42 86.36)
 		)
 		(stroke
@@
 	(wire
 		(pts
-			(xy 181.61 73.66) (xy 185.42 73.66)
+			(xy 88.9 158.75) (xy 88.9 157.48)
 		)
 		(stroke
@@
 	(wire
 		(pts
-			(xy 181.61 78.74) (xy 185.42 78.74)
+			(xy 181.61 73.66) (xy 185.42 73.66)
 		)
 		(stroke
@@
 	(wire
 		(pts
-			(xy 181.61 81.28) (xy 185.42 81.28)
-		)
-		(stroke
-			(width 0)
-			(type default)
-		)
-	)
-	(wire
-		(pts
 			(xy 125.73 114.3) (xy 139.7 114.3)
 		)
@@
 	(wire
 		(pts
-			(xy 181.61 83.82) (xy 185.42 83.82)
-		)
-		(stroke
-			(width 0)
-			(type default)
-		)
-	)
-	(wire
-		(pts
 			(xy 95.25 170.18) (xy 88.9 170.18)
 		)
@@
 	(global_label "COL 1"
 		(shape input)
-		(at 181.61 83.82 180)
+		(at 181.61 81.28 180)
 		(fields_autoplaced yes)
 		(effects
@@
 		)
 		(property "Intersheetrefs" "${INTERSHEET_REFS}"
-			(at 172.8191 83.82 0)
+			(at 172.8191 81.28 0)
 			(effects
 				(font
@@
 	(global_label "COL 0"
 		(shape input)
-		(at 181.61 86.36 180)
+		(at 181.61 78.74 180)
 		(fields_autoplaced yes)
 		(effects
@@
 		)
 		(property "Intersheetrefs" "${INTERSHEET_REFS}"
-			(at 172.8191 86.36 0)
+			(at 172.8191 78.74 0)
 			(effects
 				(font
@@
 	(global_label "COL 2"
 		(shape input)
-		(at 181.61 81.28 180)
+		(at 181.61 83.82 180)
 		(fields_autoplaced yes)
 		(effects
@@
 		)
 		(property "Intersheetrefs" "${INTERSHEET_REFS}"
-			(at 172.8191 81.28 0)
+			(at 172.8191 83.82 0)
 			(effects
 				(font
@@
 	(global_label "COL 3"
 		(shape input)
-		(at 181.61 78.74 180)
+		(at 181.61 86.36 180)
 		(fields_autoplaced yes)
 		(effects
@@
 		)
 		(property "Intersheetrefs" "${INTERSHEET_REFS}"
-			(at 172.8191 78.74 0)
+			(at 172.8191 86.36 0)
 			(effects
 				(font
@@
 			)
 		)
-		(property "Footprint" "ScottoKeebs_Components:Button_TL3342"
+		(property "Footprint" "RedComponents:SW TS-B003-Y"
 			(at 93.98 163.83 0)
 			(effects
@@
 	(symbol
 		(lib_id "Device:Battery")
-		(at 57.15 171.45 0)
+		(at 57.15 171.45 180)
 		(unit 1)
 		(exclude_from_sim no)
@@
 		(fields_autoplaced yes)
 		(property "Reference" "BT1"
-			(at 60.96 169.6084 0)
+			(at 60.96 170.7514 0)
 			(effects
 				(font
 					(size 1.27 1.27)
 				)
-				(justify left)
+				(justify right)
 			)
 		)
 		(property "Value" "Battery"
-			(at 60.96 172.1484 0)
+			(at 60.96 173.2914 0)
 			(effects
 				(font
 					(size 1.27 1.27)
 				)
-				(justify left)
+				(justify right)
 			)
 		)
-		(property "Footprint" "Connector_JST:JST_ACH_BM01B-ACHSS-A-GAN-ETF_1x01-1MP_P1.20mm_Vertical"
-			(at 57.15 169.926 90)
+		(property "Footprint" "Connector_JST:JST_EH_S2B-EH_1x02_P2.50mm_Horizontal"
+			(at 57.15 172.974 90)
 			(effects
 				(font
@@
 		)
 		(property "Datasheet" "~"
-			(at 57.15 169.926 90)
+			(at 57.15 172.974 90)
 			(effects
 				(font
